File: thesailorgps.kicad_pcb (KiCad board)
At the start: 2 copper layers, 31.7 x 29.2 mm, 56 parts, among them J1 USB_B_Micro, J2 Conn_Coaxial, J3 Conn_01x04_Male, Q1 mmbt2222a, Q2 mmbt2222a, SW1 SW_Push, U1 MCP1804x-3002xMB, U2 CH340G, U3 NEO_M8N, U4 ESP-12E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

Commit message: Improve routing
Parts:
- L1, R1, R4, U3: moved to B.Cu
- moved SW1 178.8 mm to (214.0, 134.0), turned to 90 degrees
- moved U3 178.4 mm to (200.0, 110.7), turned to 270 degrees
- moved U4 178.0 mm to (199.4, 128.0)
- moved BT1 176.2 mm to (186.7, 108.0), turned to 270 degrees
- moved R4 164.0 mm to (196.3, 101.2), turned to 270 degrees
- moved L1 159.4 mm to (195.4, 98.1), turned to 180 degrees
- moved J3 156.3 mm to (205.1, 92.9), turned to 0 degrees
- moved J2 147.8 mm to (190.5, 91.4)
- moved J1 144.7 mm to (182.6, 139.1)
- moved U5 142.8 mm to (211.9, 89.3)
- moved Q1 142.2 mm to (186.3, 116.7)
- moved Q2 142.1 mm to (186.3, 120.8)
- moved U2 139.0 mm to (183.5, 130.8), turned to 270 degrees
- moved JP3 133.2 mm to (229.2, 93.9)
- moved C2 133.1 mm to (204.8, 105.0), turned to 270 degrees
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Other:
- board size 31.7 x 29.2 mm -> 45.7 x 55.9 mm
- copper layers 2 -> 4

Commit message: Finished first routing
Parts:
- removed JP1, JP2: SolderJumper_2_Open, ronan_footprint_library:SolderJumper-2_P1.3mm_Open_RoundedPad1.0x1.5mm
- added R21: 1M, Resistors_SMD:R_0603_HandSoldering, F.Cu at (221.5, 122.4)
- added R22: 220k, Resistors_SMD:R_0603_HandSoldering, F.Cu at (219.8, 122.4)
- added REF**: MountingHole_3.2mm_M3, Mounting_Holes:MountingHole_3.2mm_M3, F.Cu at (185.1, 124.8)
- added REF**: MountingHole_3.2mm_M3, Mounting_Holes:MountingHole_3.2mm_M3, F.Cu at (185.1, 98.8)
- added REF**: MountingHole_3.2mm_M3_ISO7380_Pad, Mounting_Holes:MountingHole_3.2mm_M3_ISO7380_Pad, F.Cu at (223.9, 138.7)
- added REF**: MountingHole_3.2mm_M3_ISO14580_Pad, Mounting_Holes:MountingHole_3.2mm_M3_ISO14580_Pad, F.Cu at (174.9, 138.5)
- added REF**: MountingHole_3.2mm_M3_ISO7380_Pad, Mounting_Holes:MountingHole_3.2mm_M3_ISO7380_Pad, F.Cu at (175.4, 90.0)
- added REF**: MountingHole_3.2mm_M3_ISO14580_Pad, Mounting_Holes:MountingHole_3.2mm_M3_ISO14580_Pad, F.Cu at (223.7, 90.0)
- added REF**: MountingHole_3.2mm_M3, Mounting_Holes:MountingHole_3.2mm_M3, F.Cu at (213.6, 124.8)
- added REF**: MountingHole_3.2mm_M3, Mounting_Holes:MountingHole_3.2mm_M3, F.Cu at (213.6, 98.8)
- R1: moved to F.Cu
- moved D4 110.9 mm to (222.3, 116.6), turned to 270 degrees
- moved R3 109.5 mm to (214.8, 112.6), turned to 270 degrees
- moved C15 104.7 mm to (211.6, 118.5), turned to 90 degrees
- moved C3 100.8 mm to (207.9, 112.6), turned to 90 degrees
- moved R6 100.1 mm to (188.4, 137.3), turned to 180 degrees
- moved R8 97.1 mm to (200.1, 112.6), turned to 270 degrees
- moved R14 96.4 mm to (190.0, 123.4), turned to 270 degrees
- moved C11 92.3 mm to (183.8, 136.1)
- moved C16 92.1 mm to (181.1, 137.2), turned to 270 degrees
- moved C13 88.9 mm to (181.1, 133.4), turned to 270 degrees
- moved C12 87.7 mm to (196.8, 111.7), turned to 90 degrees
- moved C10 84.1 mm to (194.9, 105.6)
- moved C9 83.4 mm to (194.9, 107.2)
- moved R10 81.0 mm to (191.2, 88.6)
- moved R7 79.4 mm to (174.6, 122.6), turned to 90 degrees
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Connections:
- U4 pad 11: /ACC_INT -> Net-(U4-Pad11)
- U4 pad 12: /FSYNC -> Net-(U4-Pad12)
- U4 pad 2: Net-(U4-Pad2) -> /V_BATTERY_ADC
Routing:
- net +3V3: track 0.00 -> 203.1 mm, vias 0 -> 15
- net GND: track 15.2 -> 98.3 mm, vias 3 -> 184
- net /V_BACKUP: track 0.00 -> 66.7 mm, vias 0 -> 1
- net /ESP_RST: track 0.00 -> 56.4 mm
- net /SCL: track 0.00 -> 56.2 mm, vias 0 -> 2
- net /SDA: track 0.00 -> 55.9 mm
- net +5V: track 0.00 -> 54.2 mm, vias 0 -> 4
- net Net-(R6-Pad2): track 0.00 -> 51.1 mm
- net Net-(R5-Pad2): track 0.00 -> 50.0 mm
- net /RESET_GPS: track 0.00 -> 39.4 mm, vias 0 -> 1
- net Net-(R19-Pad1): track 0.00 -> 29.3 mm, vias 0 -> 1
- net /GPIO0: track 0.00 -> 26.8 mm
- net Net-(J1-Pad3): track 0.00 -> 26.2 mm
- net Net-(J1-Pad2): track 0.00 -> 23.9 mm
- net /V_BATTERY_ADC: track 0.00 -> 19.5 mm, vias 0 -> 2
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- added copper zone on B.Cu, net +3V3
- added copper zone on F.Cu, net +3V3
- added copper zone on F.Cu, net +5V
- added copper zone on B.Cu, net GND
- added copper zone on F.Cu, net GND
Other:
- board size 45.7 x 55.9 mm -> 56.4 x 55.9 mm
- copper layers 4 -> 2
- net class Default: clearance 0.2 -> 0.16
- rule trace_clearance: 0.2 -> 0.16
- rule trace_min: 0.2 -> 0.16
