File: thesailorgps.sch (KiCad schematic (older format))
At the start: 58 parts, among them J1 USB_B_Micro, J2 Conn_Coaxial, J3 Conn_01x04_Male, Q1 S8050, Q2 S8050, SW1 SW_Push, U1 SPX3819M5-L-3-3, U2 CH340G, U3 NEO_M8N, U4 ESP-12E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

Commit message: Finished schem and started routing
Parts:
- removed C6: 470pF, symbol Device:C
- removed TP1: TestPoint, symbol Connector:TestPoint
- removed U1: SPX3819M5-L-3-3, Package_TO_SOT_SMD:SOT-23-5, symbol Regulator_Linear:SPX3819M5-L-3-3
- added U1: MCP1804x-3002xMB, TO_SOT_Packages_SMD:SOT-89-3_Handsoldering, symbol Regulator_Linear:MCP1804x-3002xMB
- BT1: renamed from BT?; footprint (none) -> ronan_footprint_library:2998
- C1, C10, C11, C12, C13, C14, C15, C16, C3, C4, C5, C7, C9: footprint (none) -> Capacitors_SMD:C_0603_HandSoldering
- C2: renamed from C?; footprint (none) -> Capacitors_SMD:C_0603_HandSoldering
- C8: value 10uF -> 1uF; footprint (none) -> Capacitors_SMD:C_0603_HandSoldering
- D1: footprint (none) -> Diodes_SMD:D_0603
- D2: footprint (none) -> LEDs:LED_0603_HandSoldering
- D3: renamed from D?; footprint (none) -> LEDs:LED_0603_HandSoldering
- D4: renamed from D?; footprint (none) -> Diodes_SMD:D_0603
- J1: footprint (none) -> 105017-1001:MOLEX_105017-1001
- J2: footprint (none) -> ronan_footprint_library:SMA_coude
- J3: footprint (none) -> Connectors_Molex:Molex_PicoBlade_53261-0471_04x1.25mm_Angled
- JP1, JP2, JP3: footprint (none) -> ronan_footprint_library:SolderJumper-2_P1.3mm_Open_RoundedPad1.0x1.5mm
- L1: renamed from L?; footprint (none) -> Inductors_SMD:L_0805_HandSoldering
- Q1, Q2: value S8050 -> mmbt2222a; footprint Package_TO_SOT_THT:TO-92_Inline -> digikey-footprints:SOT-23-3
- R1, R10, R11, R12, R13, R14, R15, R16, R17, R18, R2, R3, R4, R5, R6, R7, R8, R9: footprint (none) -> Resistors_SMD:R_0603_HandSoldering
- R19, R20: renamed from R?; footprint (none) -> Resistors_SMD:R_0603_HandSoldering
- SW1: footprint (none) -> ronan_footprint_library:ebay_smd_button
- U2: footprint Package_SO:SOIC-16_3.9x9.9mm_P1.27mm -> Housings_SOIC:SOIC-16_3.9x9.9mm_Pitch1.27mm
- U3: footprint (none) -> ronan_footprint_library:neo_m8n
- U4: footprint RF_Module:ESP-12E -> RF_Modules:ESP-12E
- U5: footprint Sensor_Motion:InvenSense_QFN-24_3x3mm_P0.4mm -> digikey-footprints:QFN-24-1EP_3x3mm
- Y1: footprint (none) -> Crystals:Crystal_SMD_0603-2pin_6.0x3.5mm_HandSoldering
Connections:
- net +3V3: now also U1.1 (OUT)
- net +5V: now also U1.3 (IN)
- net GND: now also U1.2 (GND); no longer J1.6 (Shield)
- no-connect marks 4 -> 19

Commit message: Finished first routing
Parts:
- removed JP1, JP2: SolderJumper_2_Open, ronan_footprint_library:SolderJumper-2_P1.3mm_Open_RoundedPad1.0x1.5mm, symbol Jumper:SolderJumper_2_Open
- added R21: 1M, Resistors_SMD:R_0603_HandSoldering, symbol Device:R
- added R22: 220k, Resistors_SMD:R_0603_HandSoldering, symbol Device:R
Connections:
- net ACC_INT: no longer U4.11 (GPIO9)
- net FSYNC: no longer U4.12 (GPIO10)
- net GND: now also J1.6 (Shield), R22.2
- net V_BACKUP: now also R21.1
- net V_BATTERY_ADC: now reaches U4.2 (ADC)
- net V_BATTERY_ADC: now also R21.2, R22.1
- no-connect marks 19 -> 21
Other:
- note removed: "A placer près \nde la pin 10\n"
- moved on the sheet: C12, J3
Changed lines of the file:
@@
 L Connector:Conn_01x04_Male J3
 U 1 1 5BE82DDB
-P 5100 3750
-F 0 "J3" H 5206 4028 50  0000 C CNN
-F 1 "Conn_01x04_Male" H 5206 3937 50  0000 C CNN
-F 2 "Connectors_Molex:Molex_PicoBlade_53261-0471_04x1.25mm_Angled" H 5100 3750 50  0001 C CNN
-F 3 "~" H 5100 3750 50  0001 C CNN
-	1    5100 3750
-	1    0    0    -1
-$EndComp
-Text Notes 5100 3300 0    50   ~ 0
+P 4450 3750
+F 0 "J3" H 4556 4028 50  0000 C CNN
+F 1 "Conn_01x04_Male" H 4556 3937 50  0000 C CNN
+F 2 "Connectors_Molex:Molex_PicoBlade_53261-0471_04x1.25mm_Angled" H 4450 3750 50  0001 C CNN
+F 3 "~" H 4450 3750 50  0001 C CNN
+	1    4450 3750
+	1    0    0    -1
+$EndComp
+Text Notes 4450 3300 0    50   ~ 0
 SCREEN
 Wire Wire Line
@@
 $EndComp
 Wire Wire Line
-	5300 3650 5750 3650
-Wire Wire Line
-	5300 3850 5750 3850
-Wire Wire Line
-	5300 3950 5750 3950
-Text Label 5750 3950 2    50   ~ 0
+	4650 3650 5100 3650
+Wire Wire Line
+	4650 3850 5100 3850
+Wire Wire Line
+	4650 3950 5100 3950
+Text Label 5100 3950 2    50   ~ 0
 SDA
-Text Label 5750 3850 2    50   ~ 0
+Text Label 5100 3850 2    50   ~ 0
 SCL
 Wire Wire Line
-	6000 3750 6000 3550
-Wire Wire Line
-	5300 3750 6000 3750
+	5350 3750 5350 3550
+Wire Wire Line
+	4650 3750 5350 3750
 $Comp
 L power:+3V3 #PWR026
 U 1 1 5BF172A0
-P 6000 3550
-F 0 "#PWR026" H 6000 3400 50  0001 C CNN
-F 1 "+3V3" H 6015 3723 50  0000 C CNN
-F 2 "" H 6000 3550 50  0001 C CNN
-F 3 "" H 6000 3550 50  0001 C CNN
-	1    6000 3550
-	1    0    0    -1
-$EndComp
-Wire Wire Line
-	5750 3650 5750 3500
-Wire Wire Line
-	5750 3500 5850 3500
-Wire Wire Line
-	5850 3500 5850 3550
+P 5350 3550
+F 0 "#PWR026" H 5350 3400 50  0001 C CNN
+F 1 "+3V3" H 5365 3723 50  0000 C CNN
+F 2 "" H 5350 3550 50  0001 C CNN
+F 3 "" H 5350 3550 50  0001 C CNN
+	1    5350 3550
+	1    0    0    -1
+$EndComp
+Wire Wire Line
+	5100 3650 5100 3500
+Wire Wire Line
+	5100 3500 5200 3500
+Wire Wire Line
+	5200 3500 5200 3550
 $Comp
 L power:GND #PWR024
 U 1 1 5BF1A871
-P 5850 3550
-F 0 "#PWR024" H 5850 3300 50  0001 C CNN
-F 1 "GND" H 5900 3400 50  0000 C CNN
-F 2 "" H 5850 3550 50  0001 C CNN
-F 3 "" H 5850 3550 50  0001 C CNN
-	1    5850 3550
+P 5200 3550
+F 0 "#PWR024" H 5200 3300 50  0001 C CNN
+F 1 "GND" H 5250 3400 50  0000 C CNN
+F 2 "" H 5200 3550 50  0001 C CNN
+F 3 "" H 5200 3550 50  0001 C CNN
+	1    5200 3550
 	1    0    0    -1
 $EndComp
@@
 L power:+3V3 #PWR030
 U 1 1 5BFB789F
-P 7650 4850
-F 0 "#PWR030" H 7650 4700 50  0001 C CNN
-F 1 "+3V3" H 7665 5023 50  0000 C CNN
-F 2 "" H 7650 4850 50  0001 C CNN
-F 3 "" H 7650 4850 50  0001 C CNN
-	1    7650 4850
-	1    0    0    -1
-$EndComp
-Wire Wire Line
-	7650 4850 7650 4950
+P 5050 750
+F 0 "#PWR030" H 5050 600 50  0001 C CNN
+F 1 "+3V3" H 5065 923 50  0000 C CNN
+F 2 "" H 5050 750 50  0001 C CNN
+F 3 "" H 5050 750 50  0001 C CNN
+	1    5050 750
+	1    0    0    -1
+$EndComp
+Wire Wire Line
+	5050 750  5050 850
 $Comp
 L Device:C C12
 U 1 1 5BFB78A6
-P 7650 5100
-F 0 "C12" H 7765 5146 50  0000 L CNN
-F 1 "100nF" H 7765 5055 50  0000 L CNN
-F 2 "Capacitors_SMD:C_0603_HandSoldering" H 7688 4950 50  0001 C CNN
-F 3 "~" H 7650 5100 50  0001 C CNN
-	1    7650 5100
-	1    0    0    -1
-$EndComp
-Wire Wire Line
-	7650 5250 7650 5350
+P 5050 1000
+F 0 "C12" H 5165 1046 50  0000 L CNN
+F 1 "100nF" H 5165 955 50  0000 L CNN
+F 2 "Capacitors_SMD:C_0603_HandSoldering" H 5088 850 50  0001 C CNN
+F 3 "~" H 5050 1000 50  0001 C CNN
+	1    5050 1000
+	1    0    0    -1
+$EndComp
+Wire Wire Line
+	5050 1150 5050 1250
 $Comp
 L power:GND #PWR031
 U 1 1 5BFB78AE
-P 7650 5350
-F 0 "#PWR031" H 7650 5100 50  0001 C CNN
-F 1 "GND" H 7655 5177 50  0000 C CNN
-F 2 "" H 7650 5350 50  0001 C CNN
-F 3 "" H 7650 5350 50  0001 C CNN
-	1    7650 5350
-	1    0    0    -1
-$EndComp
-Text Notes 7750 5400 0    50   ~ 0
-A placer près \nde la pin 10\n
+P 5050 1250
+F 0 "#PWR031" H 5050 1000 50  0001 C CNN
+F 1 "GND" H 5055 1077 50  0000 C CNN
+F 2 "" H 5050 1250 50  0001 C CNN
+F 3 "" H 5050 1250 50  0001 C CNN
+	1    5050 1250
+	1    0    0    -1
+$EndComp
 $Comp
 L power:+3V3 #PWR032
@@
 Text Label 8500 5400 0    50   ~ 0
 FSYNC
-Wire Wire Line
-	8850 2700 8200 2700
-Text Label 8200 2700 0    50   ~ 0
-FSYNC
-Wire Wire Line
-	8850 2600 8200 2600
-Text Label 8200 2600 0    50   ~ 0
-ACC_INT
 Wire Wire Line
 	2200 6550 2350 6550
@@
 RX_GPS
 $Comp
-L Jumper:SolderJumper_2_Open JP2
-U 1 1 5C27D99A
-P 3050 1550
-F 0 "JP2" H 2950 1600 50  0000 C CNN
-F 1 "SolderJumper_2_Open" H 3050 1664 50  0001 C CNN
-F 2 "ronan_footprint_library:SolderJumper-2_P1.3mm_Open_RoundedPad1.0x1.5mm" H 3050 1550 50  0001 C CNN
-F 3 "~" H 3050 1550 50  0001 C CNN
-	1    3050 1550
-	1    0    0    -1
-$EndComp
-$Comp
-L Jumper:SolderJumper_2_Open JP1
-U 1 1 5C27DEA7
-P 2650 1650
-F 0 "JP1" H 2500 1700 50  0000 C CNN
-F 1 "SolderJumper_2_Open" H 2650 1764 50  0001 C CNN
-F 2 "ronan_footprint_library:SolderJumper-2_P1.3mm_Open_RoundedPad1.0x1.5mm" H 2650 1650 50  0001 C CNN
-F 3 "~" H 2650 1650 50  0001 C CNN
-	1    2650 1650
-	1    0    0    -1
-$EndComp
-Wire Wire Line
-	3200 1550 3250 1550
-Wire Wire Line
-	2900 1550 2100 1550
-Text Label 2100 1550 0    50   ~ 0
-SDA
-Text Label 2100 1650 0    50   ~ 0
-SCL
-Wire Wire Line
-	2800 1650 3250 1650
-Wire Wire Line
-	2500 1650 2100 1650
-$Comp
 L Connector:Conn_Coaxial J2
 U 1 1 5C308BDD
@@
 	1    0    0    -1
 $EndComp
-NoConn ~ 8850 2200
 NoConn ~ 8850 2400
 NoConn ~ 8850 2500
@@
 	1    0    0    -1
 $EndComp
-Entry Wire Line
-	4600 2750 4700 2850
-Wire Wire Line
-	1250 6450 1250 6650
+Wire Wire Line
+	1250 6450 1250 6550
+$Comp
+L Device:R R21
+U 1 1 5BF3CE63
+P 5900 3200
+F 0 "R21" H 5970 3246 50  0000 L CNN
+F 1 "1M" H 5970 3155 50  0000 L CNN
+F 2 "Resistors_SMD:R_0603_HandSoldering" V 5830 3200 50  0001 C CNN
+F 3 "~" H 5900 3200 50  0001 C CNN
+	1    5900 3200
+	1    0    0    -1
+$EndComp
+$Comp
+L Device:R R22
+U 1 1 5BF3D182
+P 5900 3700
+F 0 "R22" H 5970 3746 50  0000 L CNN
+F 1 "220k" H 5970 3655 50  0000 L CNN
+F 2 "Resistors_SMD:R_0603_HandSoldering" V 5830 3700 50  0001 C CNN
+F 3 "~" H 5900 3700 50  0001 C CNN
+	1    5900 3700
+	1    0    0    -1
+$EndComp
+Wire Wire Line
+	5900 3350 5900 3450
+Wire Wire Line
+	5900 3450 6700 3450
+Connection ~ 5900 3450
+Wire Wire Line
+	5900 3450 5900 3550
+Wire Wire Line
+	5900 3050 5900 2950
+Wire Wire Line
+	5900 2950 6700 2950
+Wire Wire Line
+	5900 3850 5900 3950
+$Comp
+L power:GND #PWR0101
+U 1 1 5BF6BA0E
+P 5900 3950
+F 0 "#PWR0101" H 5900 3700 50  0001 C CNN
+F 1 "GND" H 5905 3777 50  0000 C CNN
+F 2 "" H 5900 3950 50  0001 C CNN
+F 3 "" H 5900 3950 50  0001 C CNN
+	1    5900 3950
+	1    0    0    -1
+$EndComp
+Text Label 6700 2950 2    50   ~ 0
+V_BACKUP
+Text Label 6700 3450 2    50   ~ 0
+V_BATTERY_ADC
+Wire Wire Line
+	8850 2200 8200 2200
+Text Label 8200 2200 0    50   ~ 0
+V_BATTERY_ADC
+NoConn ~ 8850 2600
+NoConn ~ 8850 2700
+NoConn ~ 1300 2500
+Wire Wire Line
+	1150 6450 1150 6550
+Wire Wire Line
+	1150 6550 1250 6550
+Connection ~ 1250 6550
+Wire Wire Line
+	1250 6550 1250 6650
 $EndSCHEMATC
